Commit message: Added code to implement spatially and temporally varying 3D wind fields. Added model for UNC Charlotte engineering campus. Implemented draft version of visual plugin to show the wind magnitude and direction visually in gazebo.

File: xacro/iris.xacro (robot description, xacro)
@@ -136,4 +136,53 @@
     <xacro:insert_block name="rotor_inertia" />
   </xacro:vertical_rotor>
+    <gazebo>
+      <link name='/vis_body'>
+        <inertial>
+          <mass>1e-9</mass>
+          <inertia>
+            <ixx>1e-9</ixx>
+            <ixy>0</ixy>
+            <ixz>0</ixz>
+            <iyy>1e-9</iyy>
+            <iyz>0</iyz>
+            <izz>1e-9</izz>
+          </inertia>
+          <pose>0 0 0.0 0 -0 0</pose>
+        </inertial>
+        <collision name='collision'>
+          <geometry>
+            <sphere>
+              <radius>0.001</radius>
+            </sphere>
+          </geometry>
+        </collision>
+        <visual name='visual'>
+          <plugin name="sphere_wind3d_visual" filename="libgazebo_wind3d_visual_plugin.so"/>
+          <geometry>
+            <sphere>
+              <radius>0.001</radius>
+            </sphere>
+          </geometry>
+        </visual>
+      </link>
+    <joint name='/vis/base_joint' type='revolute'>
+      <child>/vis_body</child>
+      <parent>/base_link</parent>
+      <axis>
+        <xyz>1 0 0</xyz>
+        <limit>
+          <lower>0</lower>
+          <upper>0</upper>
+          <effort>0</effort>
+          <velocity>0</velocity>
+        </limit>
+        <dynamics>
+          <spring_reference>0</spring_reference>
+          <spring_stiffness>0</spring_stiffness>
+        </dynamics>
+        <use_parent_model_frame>1</use_parent_model_frame>
+      </axis>
+    </joint>
+  </gazebo>
   <gazebo>
       <link name='/imu_link'>

File: xacro/multirotor_base_px4.xacro (robot description, xacro)
@@ -55,8 +55,8 @@
           <xacro:unless value="${use_mesh_file}">
             <box size="${body_width} ${body_width} ${body_height}"/> <!-- [m] [m] [m] -->
-          </xacro:unless>
+         </xacro:unless>
         </geometry>
       </visual>
-      <collision>
+     <collision>
         <origin xyz="0 0 0" rpy="0 0 0" />
         <geometry>
@@ -95,5 +95,5 @@
       <visual>
         <geometry>
-          <!-- <cylinder length="0.005" radius="${radius_rotor}"/> --> <!-- [m] -->
+            <!-- <cylinder length="0.005" radius="${radius_rotor}"/> --> <!-- [m] -->
           <xacro:if value="${use_own_mesh}">
             <mesh filename="${mesh}"
@@ -114,5 +114,6 @@
     </link>
     <gazebo>
-      <plugin name="${robot_namespace}_${suffix}_motor_model" filename="libgazebo_motor_model.so">
+      <!-- <plugin name="${robot_namespace}_${suffix}_motor_model" filename="libgazebo_motor_model.so"> -->
+      <plugin name="${robot_namespace}_motor_model" filename="libgazebo_wind3d_motor_model_plugin.so">
         <robotNamespace>${robot_namespace}</robotNamespace>
         <jointName>${robot_namespace}/rotor_${motor_number}_joint</jointName>
